Commit message: gripper

File: ur_ws/src/Universal_Robots_ROS2_Driver/ur_moveit_config/srdf/ur_macro.srdf.xacro (robot description, xacro)
@@ -12,5 +12,5 @@
     <!--SUBGROUPS - Groups can also be formed by referencing to already defined group names-->
     <group name="${prefix}${name}_manipulator">
-      <chain base_link="${prefix}base_link" tip_link="${prefix}tool0" />
+      <chain base_link="${prefix}base_link" tip_link="${prefix}gripper_tcp" />
     </group>
     <!--GROUP STATES - Purpose - Define a named state for a particular group, in terms of joint values. This is useful to define states like 'folded arms'-->
@@ -76,4 +76,9 @@
     <!-- OnRobot RG2 gripper self‑collisions -->
     <disable_collisions link1="left_inner_finger" link2="right_inner_finger" reason="Gripper self-collision" />
+    <disable_collisions link1="left_outer_finger" link2="right_outer_finger" reason="Gripper self-collision" />
+    <!-- Add finger_width as a passive joint (so it appears in the Joints tab)-->
+    <passive_joints>
+      <joint name="${prefix}finger_width" />
+    </passive_joints>
   </xacro:macro>
 </robot>

Commit message: mtc joint

File: ur_ws/src/Universal_Robots_ROS2_Driver/ur_moveit_config/srdf/ur_macro.srdf.xacro (robot description, xacro)
@@ -22,5 +22,5 @@
     </group_state>
     <group_state name="open" group="${prefix}ur_onrobot_gripper">
-      <joint name="finger_width" value="0.100"/>
+      <joint name="finger_width" value="0.11"/>
     </group_state>
     <group_state name="${prefix}home" group="${prefix}ur_manipulator">
@@ -49,4 +49,5 @@
     </group_state>
     <!--END EFFECTOR - Purpose - Represent information about an end effector.-->
+    <end_effector name="${prefix}ur_onrobot_gripper" parent_link="${prefix}gripper_tcp" group="${prefix}ur_onrobot_gripper" parent_group="${prefix}ur_manipulator"/>
     <!--VIRTUAL JOINT - Purpose - this element defines a virtual joint between a robot link and an external frame of reference (considered fixed with respect to the robot)-->
     <!--DISABLE COLLISIONS - By default it is assumed that any link of the robot could potentially come into collision with any other link in the robot. This tag disables collision checking between a specified pair of links. -->
@@ -85,4 +86,6 @@
     <!-- OnRobot RG2 gripper self‑collisions -->
     <disable_collisions link1="left_inner_finger" link2="right_inner_finger" reason="Gripper self-collision" />
+    <!-- Obj -->
+    <disable_collisions link1="base_link_inertia" link2="ground_plane" reason="Base on ground" />
     <!-- Add finger_width as a passive joint (so it appears in the Joints tab)-->
     <passive_joints>
