Commit message: gripper & some mtc

File: ur_ws/src/Universal_Robots_ROS2_Description/urdf/ur.urdf.xacro (robot description, xacro)
@@ -1,4 +1,4 @@
 <?xml version="1.0"?>
-<robot xmlns:xacro="http://wiki.ros.org/xacro" name="$(arg name)">
+<robot xmlns:xacro="http://wiki.ros.org/xacro" name="ur">
   <!-- robot name parameter -->
   <xacro:arg name="name" default="ur"/>

File: ur_ws/src/Universal_Robots_ROS2_Driver/ur_moveit_config/srdf/ur_macro.srdf.xacro (robot description, xacro)
@@ -11,9 +11,18 @@
     <!--CHAINS - When a chain is specified, all the links along the chain (including endpoints) are included in the group. Additionally, all the joints that are parents to included links are also included. This means that joints along the chain and the parent joint of the base link are included in the group-->
     <!--SUBGROUPS - Groups can also be formed by referencing to already defined group names-->
-    <group name="${prefix}${name}_manipulator">
+    <group name="${prefix}ur_manipulator">
       <chain base_link="${prefix}base_link" tip_link="${prefix}gripper_tcp" />
     </group>
+    <group name="${prefix}ur_onrobot_gripper">
+      <joint name="finger_width" />
+    </group>
     <!--GROUP STATES - Purpose - Define a named state for a particular group, in terms of joint values. This is useful to define states like 'folded arms'-->
-    <group_state name="${prefix}home" group="${prefix}${name}_manipulator">
+    <group_state name="closed" group="${prefix}ur_onrobot_gripper">
+      <joint name="finger_width" value="0.0"/>
+    </group_state>
+    <group_state name="open" group="${prefix}ur_onrobot_gripper">
+      <joint name="finger_width" value="0.100"/>
+    </group_state>
+    <group_state name="${prefix}home" group="${prefix}ur_manipulator">
       <joint name="${prefix}elbow_joint" value="0" />
       <joint name="${prefix}shoulder_lift_joint" value="-1.5707" />
@@ -23,5 +32,5 @@
       <joint name="${prefix}wrist_3_joint" value="0" />
     </group_state>
-    <group_state name="${prefix}up" group="${prefix}${name}_manipulator">
+    <group_state name="${prefix}up" group="${prefix}ur_manipulator">
       <joint name="${prefix}elbow_joint" value="0" />
       <joint name="${prefix}shoulder_lift_joint" value="-1.5707" />
@@ -31,5 +40,5 @@
       <joint name="${prefix}wrist_3_joint" value="0" />
     </group_state>
-    <group_state name="${prefix}test_configuration" group="${prefix}${name}_manipulator">
+    <group_state name="${prefix}test_configuration" group="${prefix}ur_manipulator">
       <joint name="${prefix}elbow_joint" value="1.4" />
       <joint name="${prefix}shoulder_lift_joint" value="-1.62" />
@@ -76,5 +85,4 @@
     <!-- OnRobot RG2 gripper self‑collisions -->
     <disable_collisions link1="left_inner_finger" link2="right_inner_finger" reason="Gripper self-collision" />
-    <disable_collisions link1="left_outer_finger" link2="right_outer_finger" reason="Gripper self-collision" />
     <!-- Add finger_width as a passive joint (so it appears in the Joints tab)-->
     <passive_joints>

Commit message: srdf urdf fixes & kinematics fixes

File: ur_ws/src/Universal_Robots_ROS2_Description/urdf/ur.urdf.xacro (robot description, xacro)
@@ -6,5 +6,5 @@
   <xacro:include filename="$(find ur_description)/urdf/ur_macro.xacro"/>
   <!-- possible 'ur_type' values: ur3, ur5, ur10, ur3e, ur5e, ur7e, ur10e, ur12e, ur16e, ur8long, ur15, ur18, ur20, ur30 -->
-  <xacro:arg name="ur_type" default="ur5x"/>
+  <xacro:arg name="ur_type" default="ur3"/>
   <!-- parameters -->
   <xacro:arg name="tf_prefix" default="" />

File: ur_ws/src/Universal_Robots_ROS2_Driver/ur_moveit_config/srdf/ur_macro.srdf.xacro (robot description, xacro)
@@ -11,9 +11,21 @@
     <!--CHAINS - When a chain is specified, all the links along the chain (including endpoints) are included in the group. Additionally, all the joints that are parents to included links are also included. This means that joints along the chain and the parent joint of the base link are included in the group-->
     <!--SUBGROUPS - Groups can also be formed by referencing to already defined group names-->
+    <group name="${prefix}ur_onrobot_gripper">
+      <link name="${prefix}onrobot_base_link"/>
+      <link name="${prefix}cable_connector_0"/>
+      <link name="${prefix}cable_connector_1"/>
+      <link name="${prefix}left_inner_knuckle"/>
+      <link name="${prefix}left_outer_knuckle"/>
+      <link name="${prefix}left_inner_finger"/>
+      <link name="${prefix}left_finger_tip"/>
+      <link name="${prefix}right_inner_knuckle"/>
+      <link name="${prefix}right_outer_knuckle"/>
+      <link name="${prefix}right_inner_finger"/>
+      <link name="${prefix}right_finger_tip"/>
+      <link name="${prefix}finger_width_mock_link"/>
+      <link name="${prefix}gripper_tcp"/>
+    </group>
     <group name="${prefix}ur_manipulator">
       <chain base_link="${prefix}base_link" tip_link="${prefix}gripper_tcp" />
-    </group>
-    <group name="${prefix}ur_onrobot_gripper">
-      <joint name="finger_width" />
     </group>
     <!--GROUP STATES - Purpose - Define a named state for a particular group, in terms of joint values. This is useful to define states like 'folded arms'-->
@@ -64,32 +76,69 @@
     <disable_collisions link1="${prefix}wrist_2_link" link2="${prefix}wrist_3_link" reason="Adjacent" />
     <!-- OnRobot RG2 gripper self‑collisions -->
-    <disable_collisions link1="onrobot_base_link" link2="left_outer_knuckle" reason="Gripper self-collision" />
-    <disable_collisions link1="onrobot_base_link" link2="left_inner_knuckle" reason="Gripper self-collision" />
-    <disable_collisions link1="onrobot_base_link" link2="left_inner_finger" reason="Gripper self-collision" />
-    <disable_collisions link1="onrobot_base_link" link2="right_outer_knuckle" reason="Gripper self-collision" />
-    <disable_collisions link1="onrobot_base_link" link2="right_inner_knuckle" reason="Gripper self-collision" />
-    <disable_collisions link1="onrobot_base_link" link2="right_inner_finger" reason="Gripper self-collision" />
-    <!-- OnRobot RG2 gripper self‑collisions -->
-    <disable_collisions link1="left_outer_knuckle" link2="left_outer_knuckle" reason="Gripper self-collision" />
-    <disable_collisions link1="left_outer_knuckle" link2="left_inner_knuckle" reason="Gripper self-collision" />
-    <disable_collisions link1="left_inner_knuckle" link2="left_inner_knuckle" reason="Gripper self-collision" />
-    <disable_collisions link1="left_inner_knuckle" link2="left_inner_finger" reason="Gripper self-collision" />
-    <disable_collisions link1="left_inner_finger" link2="left_inner_finger" reason="Gripper self-collision" />
-    <disable_collisions link1="left_inner_finger" link2="left_outer_knuckle" reason="Gripper self-collision" />
-    <!-- OnRobot RG2 gripper self‑collisions -->
-    <disable_collisions link1="right_outer_knuckle" link2="right_outer_knuckle" reason="Gripper self-collision" />
-    <disable_collisions link1="right_outer_knuckle" link2="right_inner_knuckle" reason="Gripper self-collision" />
-    <disable_collisions link1="right_inner_knuckle" link2="right_inner_knuckle" reason="Gripper self-collision" />
-    <disable_collisions link1="right_inner_knuckle" link2="right_inner_finger" reason="Gripper self-collision" />
-    <disable_collisions link1="right_inner_finger" link2="right_inner_finger" reason="Gripper self-collision" />
-    <disable_collisions link1="right_inner_finger" link2="right_outer_knuckle" reason="Gripper self-collision" />
-    <!-- OnRobot RG2 gripper self‑collisions -->
-    <disable_collisions link1="left_inner_finger" link2="right_inner_finger" reason="Gripper self-collision" />
-    <!-- Obj -->
+    <disable_collisions link1="${prefix}cable_connector_0" link2="${prefix}cable_connector_1" reason="Never"/>
+    <disable_collisions link1="${prefix}cable_connector_0" link2="${prefix}left_inner_finger" reason="Never"/>
+    <disable_collisions link1="${prefix}cable_connector_0" link2="${prefix}left_inner_knuckle" reason="Never"/>
+    <disable_collisions link1="${prefix}cable_connector_0" link2="${prefix}left_outer_knuckle" reason="Never"/>
+    <disable_collisions link1="${prefix}cable_connector_0" link2="${prefix}onrobot_base_link" reason="Adjacent"/>
+    <disable_collisions link1="${prefix}cable_connector_0" link2="${prefix}right_inner_finger" reason="Never"/>
+    <disable_collisions link1="${prefix}cable_connector_0" link2="${prefix}right_inner_knuckle" reason="Never"/>
+    <disable_collisions link1="${prefix}cable_connector_0" link2="${prefix}right_outer_knuckle" reason="Never"/>
+    <disable_collisions link1="${prefix}cable_connector_0" link2="${prefix}wrist_1_link" reason="Never"/>
+    <disable_collisions link1="${prefix}cable_connector_0" link2="${prefix}wrist_2_link" reason="Never"/>
+    <disable_collisions link1="${prefix}cable_connector_0" link2="${prefix}wrist_3_link" reason="Default"/>
+    <disable_collisions link1="${prefix}cable_connector_1" link2="${prefix}left_inner_finger" reason="Never"/>
+    <disable_collisions link1="${prefix}cable_connector_1" link2="${prefix}left_inner_knuckle" reason="Never"/>
+    <disable_collisions link1="${prefix}cable_connector_1" link2="${prefix}left_outer_knuckle" reason="Never"/>
+    <disable_collisions link1="${prefix}cable_connector_1" link2="${prefix}onrobot_base_link" reason="Adjacent"/>
+    <disable_collisions link1="${prefix}cable_connector_1" link2="${prefix}right_inner_finger" reason="Never"/>
+    <disable_collisions link1="${prefix}cable_connector_1" link2="${prefix}right_inner_knuckle" reason="Never"/>
+    <disable_collisions link1="${prefix}cable_connector_1" link2="${prefix}right_outer_knuckle" reason="Never"/>
+    <disable_collisions link1="${prefix}cable_connector_1" link2="${prefix}wrist_1_link" reason="Never"/>
+    <disable_collisions link1="${prefix}cable_connector_1" link2="${prefix}wrist_2_link" reason="Default"/>
+    <disable_collisions link1="${prefix}cable_connector_1" link2="${prefix}wrist_3_link" reason="Default"/>
+    <disable_collisions link1="${prefix}left_inner_finger" link2="${prefix}left_inner_knuckle" reason="Default"/>
+    <disable_collisions link1="${prefix}left_inner_finger" link2="${prefix}left_outer_knuckle" reason="Adjacent"/>
+    <disable_collisions link1="${prefix}left_inner_finger" link2="${prefix}onrobot_base_link" reason="Never"/>
+    <disable_collisions link1="${prefix}left_inner_finger" link2="${prefix}right_inner_finger" reason="Default"/>
+    <disable_collisions link1="${prefix}left_inner_finger" link2="${prefix}right_inner_knuckle" reason="Never"/>
+    <disable_collisions link1="${prefix}left_inner_finger" link2="${prefix}right_outer_knuckle" reason="Never"/>
+    <disable_collisions link1="${prefix}left_inner_finger" link2="${prefix}wrist_1_link" reason="Never"/>
+    <disable_collisions link1="${prefix}left_inner_finger" link2="${prefix}wrist_2_link" reason="Never"/>
+    <disable_collisions link1="${prefix}left_inner_finger" link2="${prefix}wrist_3_link" reason="Never"/>
+    <disable_collisions link1="${prefix}left_inner_knuckle" link2="${prefix}left_outer_knuckle" reason="Default"/>
+    <disable_collisions link1="${prefix}left_inner_knuckle" link2="${prefix}onrobot_base_link" reason="Adjacent"/>
+    <disable_collisions link1="${prefix}left_inner_knuckle" link2="${prefix}right_inner_finger" reason="Never"/>
+    <disable_collisions link1="${prefix}left_inner_knuckle" link2="${prefix}right_inner_knuckle" reason="Never"/>
+    <disable_collisions link1="${prefix}left_inner_knuckle" link2="${prefix}right_outer_knuckle" reason="Never"/>
+    <disable_collisions link1="${prefix}left_inner_knuckle" link2="${prefix}wrist_1_link" reason="Never"/>
+    <disable_collisions link1="${prefix}left_inner_knuckle" link2="${prefix}wrist_2_link" reason="Never"/>
+    <disable_collisions link1="${prefix}left_inner_knuckle" link2="${prefix}wrist_3_link" reason="Never"/>
+    <disable_collisions link1="${prefix}left_outer_knuckle" link2="${prefix}onrobot_base_link" reason="Adjacent"/>
+    <disable_collisions link1="${prefix}left_outer_knuckle" link2="${prefix}right_inner_finger" reason="Never"/>
+    <disable_collisions link1="${prefix}left_outer_knuckle" link2="${prefix}right_inner_knuckle" reason="Never"/>
+    <disable_collisions link1="${prefix}left_outer_knuckle" link2="${prefix}right_outer_knuckle" reason="Never"/>
+    <disable_collisions link1="${prefix}left_outer_knuckle" link2="${prefix}wrist_1_link" reason="Never"/>
+    <disable_collisions link1="${prefix}left_outer_knuckle" link2="${prefix}wrist_2_link" reason="Never"/>
+    <disable_collisions link1="${prefix}left_outer_knuckle" link2="${prefix}wrist_3_link" reason="Never"/>
+    <disable_collisions link1="${prefix}onrobot_base_link" link2="${prefix}right_inner_finger" reason="Never"/>
+    <disable_collisions link1="${prefix}onrobot_base_link" link2="${prefix}right_inner_knuckle" reason="Adjacent"/>
+    <disable_collisions link1="${prefix}onrobot_base_link" link2="${prefix}right_outer_knuckle" reason="Adjacent"/>
+    <disable_collisions link1="${prefix}onrobot_base_link" link2="${prefix}wrist_1_link" reason="Never"/>
+    <disable_collisions link1="${prefix}onrobot_base_link" link2="${prefix}wrist_2_link" reason="Never"/>
+    <disable_collisions link1="${prefix}onrobot_base_link" link2="${prefix}wrist_3_link" reason="Adjacent"/>
+    <disable_collisions link1="${prefix}right_inner_finger" link2="${prefix}right_inner_knuckle" reason="Default"/>
+    <disable_collisions link1="${prefix}right_inner_finger" link2="${prefix}right_outer_knuckle" reason="Adjacent"/>
+    <disable_collisions link1="${prefix}right_inner_finger" link2="${prefix}wrist_1_link" reason="Never"/>
+    <disable_collisions link1="${prefix}right_inner_finger" link2="${prefix}wrist_2_link" reason="Never"/>
+    <disable_collisions link1="${prefix}right_inner_finger" link2="${prefix}wrist_3_link" reason="Never"/>
+    <disable_collisions link1="${prefix}right_inner_knuckle" link2="${prefix}right_outer_knuckle" reason="Default"/>
+    <disable_collisions link1="${prefix}right_inner_knuckle" link2="${prefix}wrist_1_link" reason="Never"/>
+    <disable_collisions link1="${prefix}right_inner_knuckle" link2="${prefix}wrist_2_link" reason="Never"/>
+    <disable_collisions link1="${prefix}right_inner_knuckle" link2="${prefix}wrist_3_link" reason="Never"/>
+    <disable_collisions link1="${prefix}right_outer_knuckle" link2="${prefix}wrist_1_link" reason="Never"/>
+    <disable_collisions link1="${prefix}right_outer_knuckle" link2="${prefix}wrist_2_link" reason="Never"/>
+    <disable_collisions link1="${prefix}right_outer_knuckle" link2="${prefix}wrist_3_link" reason="Never"/>
+    <!-- Ground Plane -->
     <disable_collisions link1="base_link_inertia" link2="ground_plane" reason="Base on ground" />
-    <!-- Add finger_width as a passive joint (so it appears in the Joints tab)-->
-    <passive_joints>
-      <joint name="${prefix}finger_width" />
-    </passive_joints>
   </xacro:macro>
 </robot>
